Commit message: updated new URDF

File: src/arm_robot/urdf/arm_robot.urdf (robot description, URDF)
Before this commit: robot arm_robot, 11 links, 10 joints
Links:
- removed link gripper_center
- removed link virtual_roll_link
- removed link virtual_yaw_link
- link base_link: mass 0.85623 -> 0.32792
- link link1: mass 0.17559 -> 0.11482
- link link2: mass 0.029075 -> 0.029045
- link link3: mass 0.077386 -> 0.077371
- link link5: mass 0.01684 -> 0.021692
- link link6: mass 0.021692 -> 0.01684
Joints:
- removed joint gripper_center_joint
- removed joint virtual_roll_joint
- removed joint virtual_yaw_joint
- joint base_joint: origin xyz=0.0 0.0 0.0 rpy=1.57 0 0 -> xyz=0.0 0.0 0.0 rpy=0 0 -0.1825
- joint joint1: axis 0 1 0 -> 0 0 1; limit lower=0 upper=3.142 effort=3 velocity=4 -> lower=0 upper=3.14 effort=100 velocity=3; origin xyz=0 0.0653 0 rpy=0 1.4664 0 -> xyz=0 0 0.10402 rpy=0 0 -2.9483
- joint joint2: axis -1 0 0 -> 1 0 0; limit lower=-1.57 upper=1.57 effort=3 velocity=4 -> lower=-1.57 upper=1.57 effort=100 velocity=3; origin xyz=0 0.0229 0.00043961 rpy=0.51193 0 3.1416 -> xyz=0 0 0.03687 rpy=0 0 0
- joint joint3: axis 0 0 1 -> 0 -1 0; limit lower=-1.57 upper=1.57 effort=3 velocity=4 -> lower=0 upper=3.14 effort=100 velocity=3; origin xyz=0 -0.075315 0.042319 rpy=1.5708 -0.51193 -1.5708 -> xyz=0.00047075 -0.0001562 0.085951 rpy=3.1416 -1.5491 1.5708
- joint joint4: axis 0 0 1 -> 1 0 0; limit lower=-1.57 upper=1.57 effort=3 velocity=4 -> lower=0 upper=3.14 effort=100 velocity=3; origin xyz=0.1181 0 0 rpy=0 0 0 -> xyz=0 0.0014 0.1181 rpy=1.5491 0 -1.5708
- joint joint5: axis 0 1 0 -> 0 0 -1; limit lower=0 upper=1.57 effort=1 velocity=4 -> lower=0 upper=1.57 effort=100 velocity=3; origin xyz=0.11993 0 0.012424 rpy=-3.1112 -0.89161 0 -> xyz=-0.013607 0.0040353 0.11993 rpy=-1.5708 0 0
- joint joint6: axis 0 1 0 -> 0 0 -1; limit lower=-1.57 upper=0 effort=1 velocity=4 -> lower=-1.57 upper=0 effort=100 velocity=3; origin xyz=0.11993 0 -0.015576 rpy=0.030391 -0.81089 -3.1416 -> xyz=0.014393 0.0040353 0.11993 rpy=-1.5708 0 0

Commit message: intermediate update on sim

File: src/arm_robot/urdf/arm_robot.urdf (robot description, URDF)
Before this commit: robot arm_robot, 8 links, 7 joints
Joints:
- joint joint3: limit lower=0 upper=3.14 effort=100 velocity=3 -> lower=-3.14 upper=0 effort=100 velocity=3
- joint joint4: limit lower=0 upper=3.14 effort=100 velocity=3 -> lower=-3.14 upper=0 effort=100 velocity=3

Commit message: Adding virtual joints for planner to work properly

File: src/arm_robot/urdf/arm_robot.urdf (robot description, URDF)
Before this commit: robot arm_robot, 8 links, 7 joints
Links:
- added link gripper_center
- added link virtual_roll_link, mass 1.0e-03; visual box size=0.001 0.001 0.001
- added link virtual_yaw_link, mass 1.0e-03; visual box size=0.001 0.001 0.001
Joints:
- added joint gripper_center_joint: type fixed, parent virtual_yaw_link, child gripper_center, origin xyz=0.0 0.0 0.0 rpy=0.0 0.0 0.0
- added joint virtual_roll_joint: type revolute, parent link4, child virtual_roll_link, origin xyz=0.0 0.0 0.2056 rpy=0 0 0, axis 1 0 0, limit lower=-3.1415 upper=3.1415 effort=54.0 velocity=4
- added joint virtual_yaw_joint: type revolute, parent virtual_roll_link, child virtual_yaw_link, origin xyz=0.0 0.0 0.0 rpy=0 0 0, axis 0 0 1, limit lower=-3.1415 upper=3.1415 effort=54.0 velocity=4

File: src/arm_robot_moveit/config/gazebo_arm_robot.urdf (robot description, URDF)
Before this commit: robot arm_robot, 8 links, 7 joints
Links:
- added link gripper_center
Joints:
- added joint gripper_center_joint: type fixed, parent link4, child gripper_center, origin xyz=0.0 0.0 0.2056 rpy=0.0 0.0 0.0
- joint joint4: limit lower=-3.14 upper=0 effort=100 velocity=3 -> lower=-3.14 upper=0.0 effort=100 velocity=3
